File: formula_slug_design_blocks_library.kicad_blocks/STM32G491KCU6.kicad_block/STM32G491KCU6.kicad_sch (KiCad schematic)
At the start: 14 parts

Commit message: change mcus
Parts:
- removed U?: STM32G441KBTx, Package_QFP:LQFP-32_7x7mm_P0.8mm, symbol MCU_ST_STM32G4:STM32G441KBTx
- added U1: STM32G491KCUx, Package_DFN_QFN:QFN-32-1EP_5x5mm_P0.5mm_EP3.45x3.45mm, symbol MCU_ST_STM32G4:STM32G491KCUx
Connections:
- net +3V3: now also U1.1 (VDD), U1.17 (VDD)
- net +3V3_A: now also U1.15 (VDDA)
- net BOOT0: now also U1.31 (PB8)
- net GND: now also U1.14 (VSSA), U1.16 (VSS), U1.32 (VSS), U1.33 (VSS)
- net NRST: now also U1.4 (PG10)
- net OSC_IN: now also U1.2 (PF0)
- net OSC_OUT: now also U1.3 (PF1)
- net STLINK_SWCLK: now also U1.24 (PA14)
- net STLINK_SWDIO: now also U1.23 (PA13)
- net STLINK_SWO: now also U1.26 (PB3)
- net VCP_UART_RX: now also U1.8 (PA3)
- net VCP_UART_TX: now also U1.7 (PA2)
Other:
- note added: "STM32G491KCU6 MCU"
- note removed: "STM32G441KBTx MCU"
